Commit message: implemented estimatedd inertial properties of power unit rotor, configured controller accordingly

File: description/macros/link_macros.urdf.xacro (robot description, xacro)
@@ -1,5 +1,5 @@
 <?xml version="1.0"?>
 <robot xmlns:xacro="http://www.ros.org/wiki/xacro">
-    <xacro:macro name="stator_link_macro" params="length width height xyz mass xc yc zc ixx ixy ixz iyy iyz izz">
+    <xacro:macro name="stator_link_macro" params="length width height mass xc yc zc ixx ixy ixz iyy iyz izz">
         <link name="stator_link">
             <visual>
@@ -10,5 +10,5 @@
                     <box size="${length} ${width} ${height}" />
                 </geometry>
-                <origin xyz="${xyz}" rpy="0 0 0" />
+                <origin xyz="0 0 ${height/2.0}" rpy="0 0 0" />
             </visual>
             <collision>
@@ -16,5 +16,5 @@
                     <box size="${length} ${width} ${height}" />
                 </geometry>
-                <origin xyz="${xyz}" rpy="0 0 0" />
+                <origin xyz="0 0 ${height/2.0}" rpy="0 0 0" />
             </collision>
             <inertial>
@@ -27,5 +27,5 @@
         </link>
     </xacro:macro>
-    <xacro:macro name="rotor_link_macro" params="d length xyz mass xc yc zc ixx ixy ixz iyy iyz izz">
+    <xacro:macro name="rotor_link_macro" params="d length mass xc yc zc ixx ixy ixz iyy iyz izz">
         <link name="rotor_link">
             <visual>
@@ -36,5 +36,5 @@
                     <cylinder radius="${d/2.0}" length="${length}" />
                 </geometry>
-                <origin xyz="${xyz}" rpy="0 0 0" />
+                <origin xyz="0 0 ${body_h + length/2.0}" rpy="0 0 0" />
             </visual>
             <visual>
@@ -45,5 +45,5 @@
                     <box size="${2*d} ${d/3.0} ${length}" />
                 </geometry>
-                <origin xyz="${xyz}" rpy="0 0 0" />
+                <origin xyz="0 0 ${body_h + length/2.0}" rpy="0 0 0" />
             </visual>
             <collision>
@@ -51,12 +51,12 @@
                     <cylinder radius="${d/2.0}" length="${length}" />
                 </geometry>
-                <origin xyz="${xyz}" rpy="0 0 0" />
+                <origin xyz="0 0 ${body_h + length/2.0}" rpy="0 0 0" />
             </collision>
             <inertial>
                 <mass value="${mass}"/>
-                <origin xyz="${xc} ${yc} ${zc}" rpy="0 0 0" />
-                <inertia ixx="${ixx}" ixy="${ixy}" ixz="${ixz}"
-                                      iyy="${iyy}" iyz="${iyz}"
-                                                   izz="${izz}" />
+                <origin xyz="${xc*0.001} ${yc*0.001} ${zc*0.001}" rpy="0 0 0" />
+                <inertia ixx="${ixx*0.000001}" ixy="${ixy*0.000001}" ixz="${ixz*0.000001}"
+                                      iyy="${iyy*0.000001}" iyz="${iyz*0.000001}"
+                                                   izz="${izz*0.000001}" />
             </inertial>
         </link>

File: description/power_unit_v3.urdf.xacro (robot description, xacro)
@@ -1,5 +1,5 @@
 <?xml version="1.0"?>
 <robot name="power_unit_v3" xmlns:xacro="http://www.ros.org/wiki/xacro">
-    <xacro:include filename="ros2_control.urdf.xacro" />
+    <xacro:include filename="ros2_control/ros2_control.urdf.xacro" />
     <xacro:include filename="macros/link_macros.urdf.xacro" />
     <xacro:property name="body_l" value="0.1" />
@@ -11,7 +11,6 @@
     <xacro:stator_link_macro
         length="${body_l}" width="${body_w}" height="${body_h}"
-        xyz="0 0 0"
         mass="10.0"
-        xc="0" yc="0" zc="0"
+        xc="0" yc="0" zc="${body_h/2.0}"
         ixx="${0.17}"  ixy="${0.0}"  ixz="${0.0}"
                        iyy="${0.22}" iyz="${0.0}"
@@ -19,10 +18,9 @@
     <xacro:rotor_link_macro
         d="${shaft_d}" length="${shaft_h}"
-        xyz="0 0 ${shaft_h/2.0}"
-        mass="1.0"
-        xc="0.0" yc="0.0" zc="0.0"
-        ixx="0.0225" ixy="0.0" ixz="0.0"
-                     iyy="0.0225"    iyz="0.0"
-                               izz="0.0225" />
+        mass="0.585"
+        xc="0.0" yc="0.0" zc="47.721"
+        ixx="496.884" ixy="0.0" ixz="0.0"
+                     iyy="496.884"    iyz="0.0"
+                               izz="535.230" />
     <joint name="base_joint" type="fixed">
         <parent link="base_link" />
@@ -33,5 +31,5 @@
         <parent link="stator_link" />
         <child link="rotor_link" />
-        <origin xyz="0 0 ${body_h/2.0}" rpy="0 0 0" />
+        <origin xyz="0 0 0" rpy="0 0 0" />
         <axis xyz="0 0 1" />
     </joint>

File: description/ros2_control/ros2_control_macros.urdf.xacro (robot description, xacro)
@@ -3,5 +3,4 @@
     <xacro:macro name="ros2_control_joint_macro" params="name pos_min pos_max vel_max eff_max">
         <joint name="${name}_joint">
-          <!-- co jesli joint continuous? -->
             <command_interface name="position">
               <param name="min">${pos_min}</param>
@@ -13,11 +12,7 @@
             </command_interface>
             <command_interface name="effort">
-              <param name="min">${-100000}</param>
-              <param name="max">${100000}</param>
+              <param name="min">${-eff_max}</param>
+              <param name="max">${eff_max}</param>
             </command_interface>
-            <!-- <command_interface name="effort">
-              <param name="min">${-eff_max/actuator_reduction}</param>
-              <param name="max">${eff_max/actuator_reduction}</param>
-            </command_interface> -->
             <state_interface name="position" />
             <state_interface name="velocity"/>

Commit message: fixed trapezoidal motion, added required ros2 parameters

File: description/macros/link_macros.urdf.xacro (robot description, xacro)
@@ -36,5 +36,5 @@
                     <cylinder radius="${d/2.0}" length="${length}" />
                 </geometry>
-                <origin xyz="0 0 ${body_h + length/2.0}" rpy="0 0 0" />
+                <origin xyz="0 0 ${length/2}" rpy="0 0 0" />
             </visual>
             <visual>
@@ -45,5 +45,5 @@
                     <box size="${2*d} ${d/3.0} ${length}" />
                 </geometry>
-                <origin xyz="0 0 ${body_h + length/2.0}" rpy="0 0 0" />
+                <origin xyz="0 0 ${length/2}" rpy="0 0 0" />
             </visual>
             <collision>
@@ -51,5 +51,5 @@
                     <cylinder radius="${d/2.0}" length="${length}" />
                 </geometry>
-                <origin xyz="0 0 ${body_h + length/2.0}" rpy="0 0 0" />
+                <origin xyz="0 0 ${length/2}" rpy="0 0 0" />
             </collision>
             <inertial>

File: description/power_unit_v3.urdf.xacro (robot description, xacro)
@@ -21,8 +21,8 @@
         d="${shaft_d}" length="${shaft_h}"
         mass="0.585"
-        xc="0.0" yc="0.0" zc="47.721"
-        ixx="496.884" ixy="0.0" ixz="0.0"
-                     iyy="496.884"    iyz="0.0"
-                               izz="535.230" />
+        xc="0.0" yc="0.0" zc="11.664"
+        ixx="56.082" ixy="0.0" ixz="0.0"
+                     iyy="56.082"    iyz="0.0"
+                               izz="105.479" />
     <joint name="base_joint" type="fixed">
         <parent link="world" />
@@ -33,5 +33,5 @@
         <parent link="stator_link" />
         <child link="rotor_link" />
-        <origin xyz="0 0 0" rpy="0 0 0" />
+        <origin xyz="0 0 ${body_h}" rpy="0 0 0" />
         <limit lower="${-1000*pi}" upper="${1000*pi}" effort="${motor_max_torque*reduction}" velocity="${motor_max_vel*pi/30/reduction}" />
         <axis xyz="0 0 1" />
