Commit message: fixed tags

File: description/power_unit_v3.urdf.xacro (robot description, xacro)
@@ -3,4 +3,6 @@
     <xacro:include filename="ros2_control/ros2_control.urdf.xacro" />
     <xacro:include filename="macros/link_macros.urdf.xacro" />
+    <xacro:include filename="gazebo/gz_properties.urdf.xacro"/>
+    <xacro:include filename="gazebo/gazebo.urdf.xacro"/>
     <xacro:property name="body_l" value="0.1" />
     <xacro:property name="body_w" value="0.1" />
@@ -8,5 +10,5 @@
     <xacro:property name="shaft_h" value="0.014" />
     <xacro:property name="shaft_d" value="0.035" />
-    <link name="base_link" />
+    <link name="world" />
     <xacro:stator_link_macro
         length="${body_l}" width="${body_w}" height="${body_h}"
@@ -24,12 +26,13 @@
                                izz="535.230" />
     <joint name="base_joint" type="fixed">
-        <parent link="base_link" />
+        <parent link="world" />
         <child link="stator_link" />
-        <origin xyz="0 0 0.2" rpy="0 0 0" />
+        <origin xyz="0 0 0.1" rpy="0 0 0" />
     </joint>
-    <joint name="shaft_joint" type="continuous">
+    <joint name="shaft_joint" type="revolute">
         <parent link="stator_link" />
         <child link="rotor_link" />
         <origin xyz="0 0 0" rpy="0 0 0" />
+        <limit lower="${-1000*pi}" upper="${1000*pi}" effort="${motor_max_torque*reduction}" velocity="${motor_max_vel*pi/30/reduction}" />
         <axis xyz="0 0 1" />
     </joint>

Commit message: added optimisation files

File: description/power_unit_v3.urdf.xacro (robot description, xacro)
@@ -1,8 +1,7 @@
-<?xml version="1.0"?>
-<robot name="power_unit_v3" xmlns:xacro="http://www.ros.org/wiki/xacro">
+<robot xmlns:xacro="http://www.ros.org/wiki/xacro" name="power_unit_v3">
     <xacro:include filename="ros2_control/ros2_control.urdf.xacro" />
     <xacro:include filename="macros/link_macros.urdf.xacro" />
-    <xacro:include filename="gazebo/gz_properties.urdf.xacro"/>
-    <xacro:include filename="gazebo/gazebo.urdf.xacro"/>
+    <xacro:include filename="gazebo/gz_properties.urdf.xacro" />
+    <xacro:include filename="gazebo/gazebo.urdf.xacro" />
     <xacro:property name="body_l" value="0.1" />
     <xacro:property name="body_w" value="0.1" />
@@ -11,18 +10,6 @@
     <xacro:property name="shaft_d" value="0.035" />
     <link name="world" />
-    <xacro:stator_link_macro
-        length="${body_l}" width="${body_w}" height="${body_h}"
-        mass="10.0"
-        xc="0" yc="0" zc="${body_h/2.0}"
-        ixx="${0.17}"  ixy="${0.0}"  ixz="${0.0}"
-                       iyy="${0.22}" iyz="${0.0}"
-                                     izz="${0.25}" />
-    <xacro:rotor_link_macro
-        d="${shaft_d}" length="${shaft_h}"
-        mass="0.585"
-        xc="0.0" yc="0.0" zc="11.664"
-        ixx="56.082" ixy="0.0" ixz="0.0"
-                     iyy="56.082"    iyz="0.0"
-                               izz="105.479" />
+    <xacro:stator_link_macro length="${body_l}" width="${body_w}" height="${body_h}" mass="10.0" xc="0" yc="0" zc="${body_h/2.0}" ixx="${0.17}" ixy="${0.0}" ixz="${0.0}" iyy="${0.22}" iyz="${0.0}" izz="${0.25}" />
+    <xacro:rotor_link_macro d="${shaft_d}" length="${shaft_h}" mass="0.585" xc="0.0" yc="0.0" zc="11.664" ixx="56.082" ixy="0.0" ixz="0.0" iyy="56.082" iyz="0.0" izz="105.479" />
     <joint name="base_joint" type="fixed">
         <parent link="world" />
@@ -35,4 +22,5 @@
         <origin xyz="0 0 ${body_h}" rpy="0 0 0" />
         <limit lower="${-1000*pi}" upper="${1000*pi}" effort="${motor_max_torque*reduction}" velocity="${motor_max_vel*pi/30/reduction}" />
+        <dynamics friction="0.0" damping="0.0" />
         <axis xyz="0 0 1" />
     </joint>
