Commit message: added matlab optimization files

File: description/gazebo/gz_properties.urdf.xacro (robot description, xacro)
@@ -3,9 +3,8 @@
     <!-- Gazebo joint parameters -->
     <xacro:property name="implicitSpringDamper_value" value="0" />
-    <xacro:property name="springStiffness_value" value="0" />
-    <xacro:property name="springReference_value" value="0" />
-    <xacro:property name="implicitSpringDamper_value" value="0" />
-    <xacro:property name="stopErp_value" value="0" />
-    <xacro:property name="stopCfm_value" value="0" />
+    <xacro:property name="springStiffness_value" value="0.0" />
+    <xacro:property name="springReference_value" value="0.0" />
+    <xacro:property name="stopErp_value" value="0.0" />
+    <xacro:property name="stopCfm_value" value="0.0" />
     <!-- Gazebo link parameters -->
     <xacro:property name="mu1_value" value="0" />

File: description/power_unit_v3.urdf.xacro (robot description, xacro)
@@ -10,6 +10,21 @@
     <xacro:property name="shaft_d" value="0.035" />
     <link name="world" />
-    <xacro:stator_link_macro length="${body_l}" width="${body_w}" height="${body_h}" mass="10.0" xc="0" yc="0" zc="${body_h/2.0}" ixx="${0.17}" ixy="${0.0}" ixz="${0.0}" iyy="${0.22}" iyz="${0.0}" izz="${0.25}" />
-    <xacro:rotor_link_macro d="${shaft_d}" length="${shaft_h}" mass="0.585" xc="0.0" yc="0.0" zc="11.664" ixx="56.082" ixy="0.0" ixz="0.0" iyy="56.082" iyz="0.0" izz="105.479" />
+    <xacro:stator_link_macro
+    length="${body_l}"
+    width="${body_w}"
+    height="${body_h}"
+    mass="10.0"
+    xc="0" yc="0" zc="${body_h/2.0}"
+    ixx="${0.17}" ixy="${0.0}" ixz="${0.0}"
+    iyy="${0.22}" iyz="${0.0}"
+    izz="${0.25}" />
+    <xacro:rotor_link_macro
+    d="${shaft_d}"
+    length="${shaft_h}"
+    mass="0.585"
+    xc="0.0" yc="0.0" zc="11.664"
+    ixx="56.082" ixy="0.0" ixz="0.0"
+    iyy="56.082" iyz="0.0"
+    izz="105.479" />
     <joint name="base_joint" type="fixed">
         <parent link="world" />
@@ -21,5 +36,6 @@
         <child link="rotor_link" />
         <origin xyz="0 0 ${body_h}" rpy="0 0 0" />
-        <limit lower="${-1000*pi}" upper="${1000*pi}" effort="${motor_max_torque*reduction}" velocity="${motor_max_vel*pi/30/reduction}" />
+        <limit lower="${-1000*pi}" upper="${1000*pi}"
+        effort="${motor_max_torque*reduction}" velocity="${motor_max_vel*pi/30/reduction}" />
         <dynamics friction="0.0" damping="0.0" />
         <axis xyz="0 0 1" />

File: description/pwr_unit.urdf.xacro (robot description, xacro)
@@ -28,7 +28,7 @@
   </gazebo>
   <gazebo reference="shaft_joint">
-    <implicitSpringDamper>0</implicitSpringDamper>
-    <springStiffness>0.00</springStiffness>
-    <springReference>0.00</springReference>
+    <implicitSpringDamper>1</implicitSpringDamper>
+    <springStiffness>0.0</springStiffness>
+    <springReference>0.0</springReference>
     <stopErp>0.00</stopErp>
     <stopCfm>0.00</stopCfm>
@@ -101,5 +101,5 @@
     <origin rpy="0 0 0" xyz="0 0 0.086" />
     <limit effort="34.895" lower="-3141.592653589793" upper="3141.592653589793" velocity="18.906274745776084" />
-    <dynamics damping="0.00" friction="0.00" />
+    <dynamics damping="0.0" friction="0.0" />
     <axis xyz="0 0 1" />
   </joint>
